File: hardware/fx2grok-tiny/0.1/fx2grok-tiny.kicad_pcb (KiCad board)
At the start: 2 copper layers, 13 x 13 mm, 27 parts, among them IC1 CY7C68013A-56, P1 CONN_01X05, P2 CONN_01X05, U1 MICRO-USB-B-SMD, U2 MIC5504, Y1 24MHz

Commit message: fx2grok-tiny: Add warnings that version 0.1 is broken.
Other:
- board text added: "WARNING: PCB version 0.1 is unusable, don't manufacture/use!"
Changed lines of the file:
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@@
     (links 83)
     (no_connects 0)
-    (area 50.03038 32.773983 88.390762 61.842831)
+    (area 50.03038 25.3746 97.827373 61.842831)
     (thickness 0.8)
-    (drawings 24)
+    (drawings 25)
     (tracks 345)
     (zones 0)
@@
       (net 19 GND) (clearance 0.29972))
   )
+  (gr_text "WARNING: PCB version 0.1 is unusable,\ndon't manufacture/use!\n" (at 74.49566 28.6258) (layer Dwgs.User)
+    (effects (font (size 2.032 1.524) (thickness 0.3048)))
+  )
   (gr_line (start 69.58076 49.022) (end 70.39356 49.8348) (angle 90) (layer B.SilkS) (width 0.381))
