File: hardware/fx2grok-flat/0.3/fx2grok-flat.kicad_pcb (KiCad board)
At the start: 4 copper layers, 34.9 x 16 mm, 38 parts, among them IC1 CY7C68013A-56, J1 Conn, P1 pkl_USB_OTG, U1 3.3V, U2 USBLC6-2, U3 IP425x-4-TTL, U4 IP425x-4-TTL, U5 24LC00, U6 IP425x-4-TTL, X1 24MHz

Commit message: Added via stitching around the board.
Routing:
- net GND: vias 9 -> 52
- net /shield: vias 0 -> 3
Changed lines of the file:
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@@
     (thickness 1.6)
     (drawings 46)
-    (tracks 426)
+    (tracks 472)
     (zones 0)
     (modules 38)
@@
     (34 B.Paste user)
     (35 F.Paste user)
-    (36 B.SilkS user hide)
+    (36 B.SilkS user)
     (37 F.SilkS user)
     (38 B.Mask user)
@@
   (via (at 51.5 28.7) (size 0.5) (drill 0.3) (layers F.Cu B.Cu) (net 2))
   (via (at 41.3 36.05) (size 0.5) (drill 0.3) (layers F.Cu B.Cu) (net 2))
+  (via (at 23 37) (size 0.5) (drill 0.3) (layers F.Cu B.Cu) (net 2))
+  (via (at 24 37.5) (size 0.5) (drill 0.3) (layers F.Cu B.Cu) (net 2))
+  (via (at 26 37.5) (size 0.5) (drill 0.3) (layers F.Cu B.Cu) (net 2))
+  (via (at 28 37.5) (size 0.5) (drill 0.3) (layers F.Cu B.Cu) (net 2))
+  (via (at 30 37.5) (size 0.5) (drill 0.3) (layers F.Cu B.Cu) (net 2))
+  (via (at 32 37.5) (size 0.5) (drill 0.3) (layers F.Cu B.Cu) (net 2))
+  (via (at 34 37.5) (size 0.5) (drill 0.3) (layers F.Cu B.Cu) (net 2))
+  (via (at 36 37.5) (size 0.5) (drill 0.3) (layers F.Cu B.Cu) (net 2))
+  (via (at 38 37.5) (size 0.5) (drill 0.3) (layers F.Cu B.Cu) (net 2))
+  (via (at 40 37.5) (size 0.5) (drill 0.3) (layers F.Cu B.Cu) (net 2))
+  (via (at 42 37.5) (size 0.5) (drill 0.3) (layers F.Cu B.Cu) (net 2))
+  (via (at 44 37.5) (size 0.5) (drill 0.3) (layers F.Cu B.Cu) (net 2))
+  (via (at 46 37.5) (size 0.5) (drill 0.3) (layers F.Cu B.Cu) (net 2))
+  (via (at 48 37.5) (size 0.5) (drill 0.3) (layers F.Cu B.Cu) (net 2))
+  (via (at 50 37.5) (size 0.5) (drill 0.3) (layers F.Cu B.Cu) (net 2))
+  (via (at 52 37.5) (size 0.5) (drill 0.3) (layers F.Cu B.Cu) (net 2))
+  (via (at 54 37.5) (size 0.5) (drill 0.3) (layers F.Cu B.Cu) (net 2))
+  (via (at 55 37.5) (size 0.5) (drill 0.3) (layers F.Cu B.Cu) (net 2))
+  (via (at 56.5 30) (size 0.5) (drill 0.3) (layers F.Cu B.Cu) (net 2))
+  (via (at 56.5 32) (size 0.5) (drill 0.3) (layers F.Cu B.Cu) (net 2))
+  (via (at 56.5 34) (size 0.5) (drill 0.3) (layers F.Cu B.Cu) (net 2))
+  (via (at 56.5 36) (size 0.5) (drill 0.3) (layers F.Cu B.Cu) (net 2))
+  (via (at 56.5 28) (size 0.5) (drill 0.3) (layers F.Cu B.Cu) (net 2))
+  (via (at 56.6 26) (size 0.5) (drill 0.3) (layers F.Cu B.Cu) (net 2))
+  (via (at 56.6 24) (size 0.5) (drill 0.3) (layers F.Cu B.Cu) (net 2))
+  (via (at 55 22.5) (size 0.5) (drill 0.3) (layers F.Cu B.Cu) (net 2))
+  (via (at 54 22.5) (size 0.5) (drill 0.3) (layers F.Cu B.Cu) (net 2))
+  (via (at 52 22.5) (size 0.5) (drill 0.3) (layers F.Cu B.Cu) (net 2))
+  (via (at 50 22.5) (size 0.5) (drill 0.3) (layers F.Cu B.Cu) (net 2))
+  (via (at 48 22.5) (size 0.5) (drill 0.3) (layers F.Cu B.Cu) (net 2))
+  (via (at 44 22.5) (size 0.5) (drill 0.3) (layers F.Cu B.Cu) (net 2))
+  (via (at 46 22.5) (size 0.5) (drill 0.3) (layers F.Cu B.Cu) (net 2))
+  (via (at 42 22.5) (size 0.5) (drill 0.3) (layers F.Cu B.Cu) (net 2))
+  (via (at 40 22.5) (size 0.5) (drill 0.3) (layers F.Cu B.Cu) (net 2))
+  (via (at 38 22.5) (size 0.5) (drill 0.3) (layers F.Cu B.Cu) (net 2))
+  (via (at 34 22.5) (size 0.5) (drill 0.3) (layers F.Cu B.Cu) (net 2))
+  (via (at 32 22.5) (size 0.5) (drill 0.3) (layers F.Cu B.Cu) (net 2))
+  (via (at 30 22.5) (size 0.5) (drill 0.3) (layers F.Cu B.Cu) (net 2))
+  (via (at 28 22.5) (size 0.5) (drill 0.3) (layers F.Cu B.Cu) (net 2))
+  (via (at 26 22.5) (size 0.5) (drill 0.3) (layers F.Cu B.Cu) (net 2))
+  (via (at 24.7 22.5) (size 0.5) (drill 0.3) (layers F.Cu B.Cu) (net 2))
+  (via (at 23 23) (size 0.5) (drill 0.3) (layers F.Cu B.Cu) (net 2))
+  (via (at 22.5 24.5) (size 0.5) (drill 0.3) (layers F.Cu B.Cu) (net 2))
   (via (at 33.5 34.6) (size 0.5) (drill 0.3) (layers F.Cu B.Cu) (net 5))
   (segment (start 29.750002 35.15) (end 30.35 35.15) (width 0.15) (layer B.Cu) (net 5))
@@
   (segment (start 39.675999 33.300999) (end 39.675999 34.426005) (width 0.15) (layer F.Cu) (net 8))
   (segment (start 44.398022 35.298022) (end 41.051972 35.298022) (width 0.15) (layer B.Cu) (net 8))
+  (via (at 25 30) (size 0.5) (drill 0.3) (layers F.Cu B.Cu) (net 27))
+  (via (at 24.8 32.5) (size 0.5) (drill 0.3) (layers F.Cu B.Cu) (net 27))
+  (via (at 24.8 27.5) (size 0.5) (drill 0.3) (layers F.Cu B.Cu) (net 27))
   (segment (start 35.178392 34.502652) (end 35.178392 34.756684) (width 0.15) (layer B.Cu) (net 28))
   (segment (start 35.25 34.685076) (end 35.178392 34.756684) (width 0.15) (layer F.Cu) (net 28))

Commit message: Corrected board length. (was off by 0.1mm)
Parts:
- moved J1 0.10 mm to (55.5, 30.0)
Other:
- board size 34.9 x 16 mm -> 35 x 16 mm

Commit message: Updated USB ESD diode network chip footprint.
Parts:
- turned U2 to 0 degrees
Routing:
- net /USBD_N: track 9.72 -> 10.9 mm

Commit message: Added TRIG2 silkscreen designator.
Other:
- board text added: "T 2"
Changed lines of the file:
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@@
   (general
     (thickness 1.6)
-    (drawings 46)
+    (drawings 47)
     (tracks 479)
     (zones 0)
@@
     )
   )
+  (gr_text "T\n2" (at 55.5 26.1 90) (layer B.SilkS)
+    (effects (font (size 0.5 1.25) (thickness 0.125)) (justify mirror))
+  )
   (gr_text 1BitSquared (at 32.2 30 270) (layer B.SilkS)
